File: POE.kicad_sch (KiCad schematic)
At the start: 14 parts, among them J1 Conn_01x02_Male

Commit message: Prepping for possible first build...
Parts:
- added D4: LED, LED_SMD:LED_0805_2012Metric, symbol Device:LED
- added R4: ?, Resistor_SMD:R_0805_2012Metric_Pad1.20x1.40mm_HandSolder, symbol Device:R
- C1: LCSC (none) -> C7442639
- C2, C3: LCSC (none) -> C15850
- D1, D2: LCSC (none) -> C20612967
- D3: LCSC (none) -> C280379
- MOD-1: LCSC (none) -> C5380108
- R1, R2, R3: now in the parts list
- renumbered RJ1 to J1, J1 to J2
Connections:
- net GND: now also D4.1 (K)
- net Vout: now also R4.1
- new net: D4.2 (A), R4.2
Changed lines of the file:
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@@
   (title_block
     (title "POE")
-    (rev "0.2.0")
+    (rev "1.0.0")
     (company "The Nerd Mage")
     (comment 2 "With help from Austins_Creations")
@@
     )
   )
+  (global_label "Vout" (shape input) (at 135.89 172.72 180) (fields_autoplaced)
+    (effects (font (size 1.27 1.27)) (justify right))
+    (property "Intersheet References" "${INTERSHEET_REFS}" (id 0) (at 129.3645 172.6406 0)
+      (effects (font (size 1.27 1.27)) (justify right) hide)
+    )
+  )
   (global_label "Vin+" (shape input) (at 172.72 57.15 0) (fields_autoplaced)
     (effects (font (size 1.27 1.27)) (justify left))
@@
     (property "Manufacturer_Part_Number" "Ag9905LP" (id 10) (at 250.19 645.72 0)
       (effects (font (size 1.27 1.27)) (justify left top) hide)
+    )
+    (property "LCSC" "C5380108" (id 8) (at 220.98 50.8 0)
+      (effects (font (size 1.27 1.27)) hide)
     )
     (pin "1")
@@
   )
   (symbol (lib_id "Device:R") (at 223.52 111.76 0) (unit 1)
-    (in_bom no) (on_board yes) (fields_autoplaced)
+    (in_bom yes) (on_board yes) (fields_autoplaced)
     (property "Reference" "R2" (id 0) (at 226.06 110.4899 0)
       (effects (font (size 1.27 1.27)) (justify left))
@@
     (pin "9")
   )
+  (symbol (lib_id "power:GND") (at 151.13 172.72 0) (unit 1)
+    (in_bom yes) (on_board yes)
+    (property "Reference" "#PWR0102" (id 0) (at 151.13 179.07 0)
+      (effects (font (size 1.27 1.27)) hide)
+    )
+    (property "Value" "GND" (id 1) (at 151.13 176.53 0))
+    (property "Footprint" "" (id 2) (at 151.13 172.72 0)
+      (effects (font (size 1.27 1.27)) hide)
+    )
+    (property "Datasheet" "" (id 3) (at 151.13 172.72 0)
+      (effects (font (size 1.27 1.27)) hide)
+    )
+    (pin "1")
+  )
   (symbol (lib_id "Device:C") (at 55.88 135.89 0) (unit 1)
     (in_bom yes) (on_board yes) (fields_autoplaced)
@@
     )
     (property "Datasheet" "~" (id 3) (at 55.88 135.89 0)
+      (effects (font (size 1.27 1.27)) hide)
+    )
+    (property "LCSC" "C15850" (id 4) (at 55.88 135.89 0)
       (effects (font (size 1.27 1.27)) hide)
     )
@@
   (symbol (lib_id "Austins creations:RC01374") (at 180.34 116.84 0) (unit 1)
     (in_bom no) (on_board yes) (fields_autoplaced)
-    (property "Reference" "RJ1" (id 0) (at 187.96 114.9349 0)
-      (effects (font (size 1.27 1.27)) (justify left))
-    )
-    (property "Value" "RC01374" (id 1) (at 187.96 117.4749 0)
+    (property "Reference" "J1" (id 0) (at 187.96 116.2049 0)
+      (effects (font (size 1.27 1.27)) (justify left))
+    )
+    (property "Value" "RC01374" (id 1) (at 187.96 118.7449 0)
       (effects (font (size 1.27 1.27)) (justify left))
     )
@@
   )
   (symbol (lib_id "Device:R") (at 223.52 101.6 0) (unit 1)
-    (in_bom no) (on_board yes) (fields_autoplaced)
+    (in_bom yes) (on_board yes) (fields_autoplaced)
     (property "Reference" "R1" (id 0) (at 226.06 100.3299 0)
       (effects (font (size 1.27 1.27)) (justify left))
@@
   )
   (symbol (lib_id "Device:R") (at 223.52 127 0) (unit 1)
-    (in_bom no) (on_board yes) (fields_autoplaced)
+    (in_bom yes) (on_board yes) (fields_autoplaced)
     (property "Reference" "R3" (id 0) (at 226.06 125.7299 0)
       (effects (font (size 1.27 1.27)) (justify left))
@@
     (pin "1")
   )
+  (symbol (lib_id "Device:LED") (at 147.32 172.72 180) (unit 1)
+    (in_bom yes) (on_board yes) (fields_autoplaced)
+    (property "Reference" "D4" (id 0) (at 148.9075 165.1 0))
+    (property "Value" "LED" (id 1) (at 148.9075 167.64 0))
+    (property "Footprint" "LED_SMD:LED_0805_2012Metric" (id 2) (at 147.32 172.72 0)
+      (effects (font (size 1.27 1.27)) hide)
+    )
+    (property "Datasheet" "~" (id 3) (at 147.32 172.72 0)
+      (effects (font (size 1.27 1.27)) hide)
+    )
+    (pin "1")
+    (pin "2")
+  )
   (symbol (lib_id "Diode_Bridge:MB4S") (at 153.67 46.99 0) (unit 1)
     (in_bom yes) (on_board yes) (fields_autoplaced)
@@
       (effects (font (size 1.27 1.27)) hide)
     )
+    (property "LCSC" "C20612967" (id 4) (at 153.67 46.99 0)
+      (effects (font (size 1.27 1.27)) hide)
+    )
     (pin "1")
     (pin "2")
@@
     )
     (property "Datasheet" "https://diotec.com/tl_files/diotec/files/pdf/datasheets/z1sma1.pdf" (id 3) (at 168.91 74.93 0)
+      (effects (font (size 1.27 1.27)) hide)
+    )
+    (property "LCSC" "C280379" (id 4) (at 168.91 74.93 90)
       (effects (font (size 1.27 1.27)) hide)
     )
@@
     (pin "2")
   )
+  (symbol (lib_id "Device:R") (at 139.7 172.72 90) (unit 1)
+    (in_bom yes) (on_board yes) (fields_autoplaced)
+    (property "Reference" "R4" (id 0) (at 139.7 166.37 90))
+    (property "Value" "?" (id 1) (at 139.7 168.91 90))
+    (property "Footprint" "Resistor_SMD:R_0805_2012Metric_Pad1.20x1.40mm_HandSolder" (id 2) (at 139.7 174.498 90)
+      (effects (font (size 1.27 1.27)) hide)
+    )
+    (property "Datasheet" "~" (id 3) (at 139.7 172.72 0)
+      (effects (font (size 1.27 1.27)) hide)
+    )
+    (pin "1")
+    (pin "2")
+  )
   (symbol (lib_id "Connector:Conn_01x02_Male") (at 85.09 134.62 180) (unit 1)
     (in_bom yes) (on_board yes) (fields_autoplaced)
-    (property "Reference" "J1" (id 0) (at 86.36 132.0799 0)
+    (property "Reference" "J2" (id 0) (at 86.36 132.0799 0)
       (effects (font (size 1.27 1.27)) (justify right))
     )
@@
       (effects (font (size 1.27 1.27)) hide)
     )
+    (property "LCSC" "C20612967" (id 4) (at 153.67 67.31 0)
+      (effects (font (size 1.27 1.27)) hide)
+    )
     (pin "1")
     (pin "2")
@@
       (effects (font (size 1.27 1.27)) hide)
     )
+    (property "LCSC" "C7442639" (id 4) (at 29.21 135.89 0)
+      (effects (font (size 1.27 1.27)) hide)
+    )
     (pin "1")
     (pin "2")
@@
       (effects (font (size 1.27 1.27)) hide)
     )
+    (property "LCSC" "C15850" (id 4) (at 41.91 135.89 0)
+      (effects (font (size 1.27 1.27)) hide)
+    )
     (pin "1")
     (pin "2")
@@
       (reference "#PWR0101") (unit 1) (value "GND") (footprint "")
     )
+    (path "/1a7a051d-8606-4714-b0a8-b6471a497a06"
+      (reference "#PWR0102") (unit 1) (value "GND") (footprint "")
+    )
     (path "/dab3b84e-7f55-44d6-8fae-108eec6adc14"
       (reference "#PWR0105") (unit 1) (value "GND") (footprint "")
@@
       (reference "D3") (unit 1) (value "SMAJ58A") (footprint "Diode_SMD:D_SMA")
     )
+    (path "/6e032d7a-4dc4-4932-9c99-ddb2510bc012"
+      (reference "D4") (unit 1) (value "LED") (footprint "LED_SMD:LED_0805_2012Metric")
+    )
+    (path "/2fc1c0d9-0c5e-4da1-8ab1-479c27a16f8a"
+      (reference "J1") (unit 1) (value "RC01374") (footprint "tightstuff:RC01374")
+    )
     (path "/c02961b0-e06d-492c-9aa7-5f7703cff2d6"
-      (reference "J1") (unit 1) (value "Conn_01x02_Male") (footprint "Connector_PinHeader_2.54mm:PinHeader_1x02_P2.54mm_Horizontal")
+      (reference "J2") (unit 1) (value "Conn_01x02_Male") (footprint "Connector_PinHeader_2.54mm:PinHeader_1x02_P2.54mm_Horizontal")
     )
     (path "/ac28726d-d584-4b99-9a7c-579a41b6a0db"
@@
       (reference "R3") (unit 1) (value "Rmin") (footprint "Resistor_SMD:R_0805_2012Metric_Pad1.20x1.40mm_HandSolder")
     )
-    (path "/2fc1c0d9-0c5e-4da1-8ab1-479c27a16f8a"
-      (reference "RJ1") (unit 1) (value "RC01374") (footprint "tightstuff:RC01374")
+    (path "/bef42c16-28c8-4567-8d30-8f0e937a5474"
+      (reference "R4") (unit 1) (value "?") (footprint "Resistor_SMD:R_0805_2012Metric_Pad1.20x1.40mm_HandSolder")
     )
     (path "/034a4306-bd74-4c85-81e6-2f9db7c7bd59"

Commit message: gerbers produced, boards & parts ordered... (w/slow-boat shipping...)
Parts:
- J1: now in the parts list
Changed lines of the file:
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@@
       (effects (font (size 1.27 1.27)) (justify left top) hide)
     )
-    (property "LCSC" "C5380108" (id 8) (at 220.98 50.8 0)
+    (property "LCSC" "C5380108" (id 11) (at 220.98 50.8 0)
       (effects (font (size 1.27 1.27)) hide)
     )
@@
   )
   (symbol (lib_id "Austins creations:RC01374") (at 180.34 116.84 0) (unit 1)
-    (in_bom no) (on_board yes) (fields_autoplaced)
+    (in_bom yes) (on_board yes) (fields_autoplaced)
     (property "Reference" "J1" (id 0) (at 187.96 116.2049 0)
       (effects (font (size 1.27 1.27)) (justify left))
