File: POE.kicad_sch (KiCad schematic)
At the start: 16 parts, among them J1 RC01374, J2 Conn_01x02_Male

Commit message: Post-test thoughts & adjustments.
Parts:
- added Rl2: Rmin, Resistor_SMD:R_0805_2012Metric_Pad1.20x1.40mm_HandSolder, symbol Device:R
- renumbered R3 to Rl1
Connections:
- net GND: now also Rl2.2
- net Vout: now also Rl2.1
Changed lines of the file:
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@@
     (comment 2 "With help from Austins_Creations")
   )
+  (junction (at 223.52 130.81) (diameter 0) (color 0 0 0 0)
+  )
   (junction (at 55.88 132.08) (diameter 0) (color 0 0 0 0)
   )
@@
   (junction (at 168.91 81.28) (diameter 0) (color 0 0 0 0)
   )
+  (junction (at 223.52 123.19) (diameter 0) (color 0 0 0 0)
+  )
   (wire (pts (xy 218.44 106.68) (xy 223.52 106.68))
     (stroke (width 0) (type default) (color 0 0 0 0))
@@
     (stroke (width 0) (type default) (color 0 0 0 0))
   )
+  (wire (pts (xy 223.52 123.19) (xy 232.41 123.19))
+    (stroke (width 0) (type default) (color 0 0 0 0))
+  )
   (wire (pts (xy 172.72 120.65) (xy 172.72 104.14))
     (stroke (width 0) (type default) (color 0 0 0 0))
@@
   )
   (wire (pts (xy 168.91 78.74) (xy 168.91 81.28))
+    (stroke (width 0) (type default) (color 0 0 0 0))
+  )
+  (wire (pts (xy 223.52 130.81) (xy 232.41 130.81))
     (stroke (width 0) (type default) (color 0 0 0 0))
   )
@@
     (effects (font (size 5 5) (thickness 1) bold) (justify left bottom))
   )
-  (text "Minimum Load: 200mA\nDatasheet section 2.3.3" (at 234.95 128.27 0)
+  (text "Minimum Load: 200mA\nDatasheet section 2.3.3" (at 243.84 128.27 0)
     (effects (font (size 1.27 1.27)) (justify left bottom))
   )
@@
       (effects (font (size 1.27 1.27)) (justify left) hide)
     )
+  )
+  (symbol (lib_id "Device:R") (at 232.41 127 0) (unit 1)
+    (in_bom yes) (on_board yes) (fields_autoplaced)
+    (property "Reference" "Rl2" (id 0) (at 234.95 125.7299 0)
+      (effects (font (size 1.27 1.27)) (justify left))
+    )
+    (property "Value" "Rmin" (id 1) (at 234.95 128.2699 0)
+      (effects (font (size 1.27 1.27)) (justify left))
+    )
+    (property "Footprint" "Resistor_SMD:R_0805_2012Metric_Pad1.20x1.40mm_HandSolder" (id 2) (at 230.632 127 90)
+      (effects (font (size 1.27 1.27)) hide)
+    )
+    (property "Datasheet" "~" (id 3) (at 232.41 127 0)
+      (effects (font (size 1.27 1.27)) hide)
+    )
+    (pin "1")
+    (pin "2")
   )
   (symbol (lib_id "Ag9912LP:Ag9912LP") (at 220.98 50.8 0) (unit 1)
@@
   (symbol (lib_id "Device:R") (at 223.52 127 0) (unit 1)
     (in_bom yes) (on_board yes) (fields_autoplaced)
-    (property "Reference" "R3" (id 0) (at 226.06 125.7299 0)
+    (property "Reference" "Rl1" (id 0) (at 226.06 125.7299 0)
       (effects (font (size 1.27 1.27)) (justify left))
     )
@@
       (effects (font (size 1.27 1.27)) hide)
     )
-    (property "Datasheet" "https://diotec.com/tl_files/diotec/files/pdf/datasheets/z1sma1.pdf" (id 3) (at 168.91 74.93 0)
+    (property "Datasheet" "https://datasheet.lcsc.com/lcsc/1809301633_Suzhou-Good-Ark-Elec-SMAJ58A_C280379.pdf" (id 3) (at 168.91 74.93 0)
       (effects (font (size 1.27 1.27)) hide)
     )
@@
       (reference "R2") (unit 1) (value "?") (footprint "Resistor_SMD:R_0805_2012Metric_Pad1.20x1.40mm_HandSolder")
     )
-    (path "/652c9e56-d979-4354-9c89-0a279c99fcb4"
-      (reference "R3") (unit 1) (value "Rmin") (footprint "Resistor_SMD:R_0805_2012Metric_Pad1.20x1.40mm_HandSolder")
-    )
     (path "/bef42c16-28c8-4567-8d30-8f0e937a5474"
       (reference "R4") (unit 1) (value "?") (footprint "Resistor_SMD:R_0805_2012Metric_Pad1.20x1.40mm_HandSolder")
     )
+    (path "/652c9e56-d979-4354-9c89-0a279c99fcb4"
+      (reference "Rl1") (unit 1) (value "Rmin") (footprint "Resistor_SMD:R_0805_2012Metric_Pad1.20x1.40mm_HandSolder")
+    )
+    (path "/00f4b103-44b6-432e-8a96-c230b0d6b5d4"
+      (reference "Rl2") (unit 1) (value "Rmin") (footprint "Resistor_SMD:R_0805_2012Metric_Pad1.20x1.40mm_HandSolder")
+    )
     (path "/034a4306-bd74-4c85-81e6-2f9db7c7bd59"
